File: ESP8266ControllerCircuit/ESP8266ControllerCircuit.kicad_pcb (KiCad board)
At the start: 2 copper layers, 75 x 30 mm, 25 parts, among them J1 Input, J2 Input, J3 Input, J4 Input, J5 Optional, U1 WeMos_mini, U2 EL3H7(B)(TA)-G, U3 PCF8574T/3,518

Commit message: ESP8266 controller: R2 is still 4K7 in the PCB, 2K2 everywhere else
R2 pulls the ESP8266's RX line (D7) to ground, and it was dropped from 4k7 to 2k2
to fix intermittent comms errors between the controller and the modules - #59, and
the forum thread it links to:

  https://community.openenergymonitor.org/t/workaround-for-the-communication-problems-change-resistor-in-controller/16388

  "I've just swapped my board to 2.2k and no issues, so will recommend that going
   forward"

The schematic carries that: R2 is 2K2, with C17520 / 0805W8F2201T5E assigned to it
in 922e88e.  So do the netlist, the XML, the CSV and the JLCPCB BOM.  The same
change was made to the modules at the same time - ModuleV421 R16 is 4.7k, and
ModuleV440 R16 is 2.2k with that same C17520.

The PCB was never brought along.  Its footprint value has read 4K7 since the file
was renamed in daa65dd, and the two position files exported from it repeat it.

Nothing is manufactured differently by this: the value lives on F.Fab, which is not
among the plotted layers, and JLCPCB takes component values from the BOM by
designator.  It matters when reading the board - the PCB and the position files are
the only places that still name the value that caused the problem.
Parts:
- R2: value 4K7 -> 2K2
Changed lines of the file:
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@@
       (effects (font (size 1 1) (thickness 0.15)))
     )
-    (fp_text value 4K7 (at -4 0 180) (layer F.Fab)
+    (fp_text value 2K2 (at -4 0 180) (layer F.Fab)
       (effects (font (size 1 1) (thickness 0.15)))
     )
