File: ControllerCircuit/ControllerCircuit.kicad_sch (KiCad schematic)
At the start: 91 parts, among them J1 4PinBlock, J10 ESTOP, J11 19PinSocket, J12 4PinBlock, J13 14PinSocket, J14 Unused header, J15 Molex 0472192001, J16 4PinSocket, J17 4PinBlock, J2 ScrewTerminal3Pin, J3 ScrewTerminal3Pin, J4 4PinBlock, J5 ScrewTerminal, J6 19PinSocket, J7 4PinBlock, J8 2x3 2.54mm IDC Connectors, J9 4PinBlock, K1 SRD-05VDC-SL-C, K2 SRD-05VDC-SL-C, Q1 AO3400A, Q2 AO3400A, Q3 AO3401A, Q4 AO3400A, SW1 SW_Push, SW2 SW_Push, U1 TXS0102DCU, U12 LT219-1, U2 EL3H7(B)(TA)-G, U3 TCA6416APWR, U4 ESP32-DEVKITC-32D, U5 SN65HVD75DR, U6 AMS1117-3.3, U7 SN65HVD1050D, U8 INA229, U9 LT219-1

Commit message: Five parts on the controller cannot be ordered as they stand
Checked every LCSC code in this board's BOM against the JLCPCB parts API.  Three of
these are discontinued rather than merely out of stock - the parts API returns them
with "停产" in the name, so waiting will not help.

  C3,C4  22uF 6.3V tantalum  C110786  discontinued, 0 in stock
                          -> C7182    Kyocera AVX TAJA226K006RNJ, 12,926 in stock
                                      same CASE-A-3216-18 outline, same 22uF 6.3V
                                      +/-10%, same -55 to +125C

  D1     RGB LED            C219409  discontinued, 0 in stock
                          -> C784540  TCWIN TC5050RGBF08-3CJH-AF53A, 811,463 in
                                      stock, same SMD5050-6P, same discrete-diode
                                      construction, same -40 to +85C
                                      Pinout matches: anodes on 1/2/3, G 1-6,
                                      R 2-5, B 3-4, so it drops straight in
                                      Brighter on all three - 600-800/1500-2000/
                                      400-600mcd against 460/1300/270 - and its
                                      blue Vf tops out at 3.2V rather than 3.4V,
                                      which is the colour with least headroom on
                                      a 3.3V rail through 220R

  D3,D4  yellow LED         C72038   0 in stock
                          -> C89811   NationStar NCD0603Y2, 61,378 in stock, and
                                      Preferred, so it costs no setup fee
                                      Vf 1.6-2.6V against 1.7-2.3V, 586-595nm
                                      against 585-591nm, 220mcd against 90-180mcd
                                      R12 and R13 stay at 560R: these sit across
                                      the relay coils on FUSED5V, so the current
                                      does not move

  U2     EL3H7 op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
Parts:
- C3, C4: LCSCStockCode C110786 -> C7182
- D1: LCSCStockCode C219409 -> C784540
- D3, D4: LCSCStockCode C72038 -> C89811
- Q1, Q2, Q4: LCSCStockCode C344010 -> C20917
- U2: value EL3H7(B)(TA)-G -> EL3H7B; LCSCStockCode C32565 -> C41371267
Changed lines of the file:
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@@
       (effects (font (size 1.27 1.27)) hide)
     )
-    (property "Datasheet" "https://datasheet.lcsc.com/szlcsc/Hongli-Zhihui-HONGLITRONIC-HL-AF-5060H271BU46FU79GC-S1-THL_C219409.pdf" (at 83.82 68.58 0)
+    (property "Datasheet" "https://wmsc.lcsc.com/wmsc/upload/file/pdf/v2/lcsc/2307310952_TCWIN-TC5050RGBF08-3CJH-AF53A_C784540.pdf" (at 83.82 68.58 0)
       (effects (font (size 1.27 1.27)) hide)
     )
-    (property "LCSCStockCode" "C219409" (at 83.82 68.58 0)
+    (property "LCSCStockCode" "C784540" (at 83.82 68.58 0)
       (effects (font (size 1.27 1.27)) hide)
     )
@@
       (effects (font (size 1.27 1.27)))
     )
-    (property "Value" "EL3H7(B)(TA)-G" (at 165.1 16.9164 0)
+    (property "Value" "EL3H7B" (at 165.1 16.9164 0)
       (effects (font (size 1.27 1.27)))
     )
@@
       (effects (font (size 1.27 1.27) italic) (justify left) hide)
     )
-    (property "Datasheet" "https://datasheet.lcsc.com/szlcsc/Everlight-Elec-EL3H7-B-TA-G_C32565.pdf" (at 165.1 22.86 0)
+    (property "Datasheet" "https://www.lcsc.com/datasheet/lcsc_datasheet_2409021207_AOTE-EL3H7B_C41371267.pdf" (at 165.1 22.86 0)
       (effects (font (size 1.27 1.27)) (justify left) hide)
     )
-    (property "LCSCStockCode" "C32565" (at 165.1 22.86 0)
+    (property "LCSCStockCode" "C41371267" (at 165.1 22.86 0)
       (effects (font (size 1.27 1.27)) hide)
     )
@@
       (effects (font (size 1.27 1.27)) hide)
     )
-    (property "Datasheet" "https://datasheet.lcsc.com/szlcsc/Hunan-Xiangyee-in-S-T-CA45-A010M226T_C126948.pdf" (at 159.893 79.121 0)
+    (property "Datasheet" "https://www.lcsc.com/datasheet/lcsc_datasheet_2304140030_Kyocera-AVX-TAJA226K006RNJ_C7182.pdf" (at 159.893 79.121 0)
       (effects (font (size 1.27 1.27)) hide)
     )
-    (property "LCSCStockCode" "C110786" (at 159.893 79.121 0)
+    (property "LCSCStockCode" "C7182" (at 159.893 79.121 0)
       (effects (font (size 1.27 1.27)) hide)
     )
@@
       (effects (font (size 1.27 1.27)) hide)
     )
-    (property "Datasheet" "https://datasheet.lcsc.com/szlcsc/Hunan-Xiangyee-in-S-T-CA45-A010M226T_C126948.pdf" (at 180.086 79.121 0)
+    (property "Datasheet" "https://www.lcsc.com/datasheet/lcsc_datasheet_2304140030_Kyocera-AVX-TAJA226K006RNJ_C7182.pdf" (at 180.086 79.121 0)
       (effects (font (size 1.27 1.27)) hide)
     )
-    (property "LCSCStockCode" "C110786" (at 180.086 79.121 0)
+    (property "LCSCStockCode" "C7182" (at 180.086 79.121 0)
       (effects (font (size 1.27 1.27)) hide)
     )
@@
       (effects (font (size 1.27 1.27)) hide)
     )
-    (property "Datasheet" "https://datasheet.lcsc.com/lcsc/1912111437_BORN-AO3400A_C344010.pdf" (at 40.64 162.56 0)
+    (property "Datasheet" "https://www.lcsc.com/datasheet/lcsc_datasheet_1811081213_Alpha---Omega-Semicon-AO3400A_C20917.pdf" (at 40.64 162.56 0)
       (effects (font (size 1.27 1.27)) hide)
     )
-    (property "LCSCStockCode" "C344010" (at 40.64 162.56 0)
+    (property "LCSCStockCode" "C20917" (at 40.64 162.56 0)
       (effects (font (size 1.27 1.27)) hide)
     )
@@
       (effects (font (size 1.27 1.27)) hide)
     )
-    (property "Datasheet" "" (at 22.86 151.13 0)
+    (property "Datasheet" "https://www.lcsc.com/datasheet/lcsc_datasheet_2008201033_Foshan-NationStar-Optoelectronics-NCD0603Y2_C89811.pdf" (at 22.86 151.13 0)
       (effects (font (size 1.27 1.27)) hide)
     )
-    (property "LCSCStockCode" "C72038" (at 22.86 151.13 0)
+    (property "LCSCStockCode" "C89811" (at 22.86 151.13 0)
       (effects (font (size 1.27 1.27)) hide)
     )
@@
       (effects (font (size 1.27 1.27)) hide)
     )
-    (property "Datasheet" "https://datasheet.lcsc.com/lcsc/1912111437_BORN-AO3400A_C344010.pdf" (at 116.84 165.1 0)
+    (property "Datasheet" "https://www.lcsc.com/datasheet/lcsc_datasheet_1811081213_Alpha---Omega-Semicon-AO3400A_C20917.pdf" (at 116.84 165.1 0)
       (effects (font (size 1.27 1.27)) hide)
     )
-    (property "LCSCStockCode" "C344010" (at 116.84 165.1 0)
+    (property "LCSCStockCode" "C20917" (at 116.84 165.1 0)
       (effects (font (size 1.27 1.27)) hide)
     )
@@
       (effects (font (size 1.27 1.27)) hide)
     )
-    (property "Datasheet" "" (at 99.06 153.67 0)
+    (property "Datasheet" "https://www.lcsc.com/datasheet/lcsc_datasheet_2008201033_Foshan-NationStar-Optoelectronics-NCD0603Y2_C89811.pdf" (at 99.06 153.67 0)
       (effects (font (size 1.27 1.27)) hide)
     )
-    (property "LCSCStockCode" "C72038" (at 99.06 153.67 0)
+    (property "LCSCStockCode" "C89811" (at 99.06 153.67 0)
       (effects (font (size 1.27 1.27)) hide)
     )
@@
       (effects (font (size 1.27 1.27) italic) (justify left) hide)
     )
-    (property "Datasheet" "https://datasheet.lcsc.com/lcsc/1912111437_BORN-AO3400A_C344010.pdf" (at 167.64 40.64 0)
+    (property "Datasheet" "https://www.lcsc.com/datasheet/lcsc_datasheet_1811081213_Alpha---Omega-Semicon-AO3400A_C20917.pdf" (at 167.64 40.64 0)
       (effects (font (size 1.27 1.27)) (justify left) hide)
     )
-    (property "LCSCStockCode" "C344010" (at 167.64 40.64 0)
+    (property "LCSCStockCode" "C20917" (at 167.64 40.64 0)
       (effects (font (size 1.27 1.27)) hide)
     )
