File: ModuleV490-AllInOne/Module_16S.kicad_sch (KiCad schematic)
At the start: 61 parts, among them J14 BALANCE BOARD, J15 BALANCE BOARD, J6 MALE PLUG, J7 CELL CONNECTOR, U1 MAX14921ECS+T, U3 MCP33151-05-E/MS, U6 MCP1502T-45E/CHY

Commit message: V490: ten part numbers, all like-for-like
Monitor board:

  U11  AP2204K-5.0TRG1  C112031  discontinued
                     -> C5378676  AP2205-50W5-7, the Diodes successor, same
                                  SOT-23-5, same 5V/200mA
  U3   MCP33151-05     C635984  0 in stock
                     -> C627094   same part, the T is tape and reel
  U13  EL3H7           C32565   0 in stock
                     -> C41371267 AOTE EL3H7B, same CTR rank and SSOP-4
  L1   100uH           C286551  24 in stock
                     -> C76826    NLV25T-101J-PF against -EF, same 100uH 1008
  D21  SS210           C432298  Extended
                     -> C14996    same part number, Basic
  D?   1N4002W         C169542  Extended
                     -> C18199086 same part number, Preferred
  C44  33nF            C113810  786 in stock
                     -> C21117    Basic, same 33nF 0603 X7R
  C30,C31  14pF        C458857  Extended, thin stock
                     -> C1548     15pF 0402 C0G, Basic.  The only value change
                                  here: on a 8MHz crystal the shift works out
                                  around 3ppm

Balancer board:

  C0..C15  yellow LED  C72038   0 in stock
                     -> C89811    NationStar NCD0603Y2, still yellow, Preferred
  Q..      AO3400A     C347475  Extended
                     -> C20917    same part number, Basic

Nothing changes colour and nothing changes function.  The yellow LEDs stay yellow
deliberately: swapping them for red would be visible to whoever built the board, and
a board whose indicators changed colour is not the same board even if every part is
in stock.  There is a case for red - the cell modules use red for the bypass
indicator and these sixteen do the same job - but that is a revision, not a
substitution.

U6 is left alone.  MCP1502T-45E/CHY is down to 1 in stock and the obvious
replacement, REF345SOT233, is SOT-23-3 where this is SOT-23-6.  That needs the
board changing, not the BOM.  MCP1501T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
Parts:
- U3: LCSCStockCode C635984 -> C627094
Changed lines of the file:
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@@
       (effects (font (size 1.27 1.27)) hide)
     )
-    (property "LCSCStockCode" "C635984" (at 250.19 93.345 0)
+    (property "LCSCStockCode" "C627094" (at 250.19 93.345 0)
       (effects (font (size 1.27 1.27)) hide)
     )
