File: ModuleV490-AllInOne/PowerSupply.kicad_sch (KiCad schematic)
At the start: 26 parts, among them J5 POWER_IN, U10 XL7005A, U11 AP2204K-5.0TRG1, U12 XC6206-1.8NR, U9 XC6206-3.3V

Commit message: V490: ten part numbers, all like-for-like
Monitor board:

  U11  AP2204K-5.0TRG1  C112031  discontinued
                     -> C5378676  AP2205-50W5-7, the Diodes successor, same
                                  SOT-23-5, same 5V/200mA
  U3   MCP33151-05     C635984  0 in stock
                     -> C627094   same part, the T is tape and reel
  U13  EL3H7           C32565   0 in stock
                     -> C41371267 AOTE EL3H7B, same CTR rank and SSOP-4
  L1   100uH           C286551  24 in stock
                     -> C76826    NLV25T-101J-PF against -EF, same 100uH 1008
  D21  SS210           C432298  Extended
                     -> C14996    same part number, Basic
  D?   1N4002W         C169542  Extended
                     -> C18199086 same part number, Preferred
  C44  33nF            C113810  786 in stock
                     -> C21117    Basic, same 33nF 0603 X7R
  C30,C31  14pF        C458857  Extended, thin stock
                     -> C1548     15pF 0402 C0G, Basic.  The only value change
                                  here: on a 8MHz crystal the shift works out
                                  around 3ppm

Balancer board:

  C0..C15  yellow LED  C72038   0 in stock
                     -> C89811    NationStar NCD0603Y2, still yellow, Preferred
  Q..      AO3400A     C347475  Extended
                     -> C20917    same part number, Basic

Nothing changes colour and nothing changes function.  The yellow LEDs stay yellow
deliberately: swapping them for red would be visible to whoever built the board, and
a board whose indicators changed colour is not the same board even if every part is
in stock.  There is a case for red - the cell modules use red for the bypass
indicator and these sixteen do the same job - but that is a revision, not a
substitution.

U6 is left alone.  MCP1502T-45E/CHY is down to 1 in stock and the obvious
replacement, REF345SOT233, is SOT-23-3 where this is SOT-23-6.  That needs the
board changing, not the BOM.  MCP1501T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
Parts:
- C44: LCSCStockCode C113810 -> C21117; PartNumber CC0603KRX7R8BB333 -> CL10B333KB8NNNC
- D20: LCSCStockCode C169542 -> C18199086
- D21: LCSCStockCode C432298 -> C14996
- L1: LCSCStockCode C286551 -> C76826; PartNumber NLV25T-101J-EF -> NLV25T-101J-PF
- U11: value AP2204K-5.0TRG1 -> AP2205-50W5-7; LCSCStockCode C112031 -> C5378676; PartNumber AP2204K-5.0TRG1 -> AP2205-50W5-7
Changed lines of the file:
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@@
       (effects (font (size 1.27 1.27)) hide)
     )
-    (property "PartNumber" "CC0603KRX7R8BB333" (at 123.825 75.565 0)
-      (effects (font (size 1.27 1.27)) hide)
-    )
-    (property "LCSCStockCode" "C113810" (at 123.825 75.565 0)
+    (property "PartNumber" "CL10B333KB8NNNC" (at 123.825 75.565 0)
+      (effects (font (size 1.27 1.27)) hide)
+    )
+    (property "LCSCStockCode" "C21117" (at 123.825 75.565 0)
       (effects (font (size 1.27 1.27)) hide)
     )
@@
       (effects (font (size 1.27 1.27)) hide)
     )
-    (property "LCSCStockCode" "C169542" (at 41.275 73.025 0)
+    (property "LCSCStockCode" "C18199086" (at 41.275 73.025 0)
       (effects (font (size 1.27 1.27)) hide)
     )
@@
       (effects (font (size 1.27 1.27)) hide)
     )
-    (property "LCSCStockCode" "C432298" (at 95.885 76.835 0)
+    (property "LCSCStockCode" "C14996" (at 95.885 76.835 0)
       (effects (font (size 1.27 1.27)) hide)
     )
@@
       (effects (font (size 1.27 1.27)))
     )
-    (property "Value" "AP2204K-5.0TRG1" (at 210.185 34.925 0)
+    (property "Value" "AP2205-50W5-7" (at 210.185 34.925 0)
       (effects (font (size 1.27 1.27)))
     )
@@
       (effects (font (size 1.27 1.27)) hide)
     )
-    (property "PartNumber" "AP2204K-5.0TRG1" (at 210.185 40.64 0)
-      (effects (font (size 1.27 1.27)) hide)
-    )
-    (property "LCSCStockCode" "C112031" (at 210.185 40.64 0)
+    (property "PartNumber" "AP2205-50W5-7" (at 210.185 40.64 0)
+      (effects (font (size 1.27 1.27)) hide)
+    )
+    (property "LCSCStockCode" "C5378676" (at 210.185 40.64 0)
       (effects (font (size 1.27 1.27)) hide)
     )
@@
       (effects (font (size 1.27 1.27)) hide)
     )
-    (property "PartNumber" "NLV25T-101J-EF" (at 106.68 73.025 0)
-      (effects (font (size 1.27 1.27)) hide)
-    )
-    (property "LCSCStockCode" "C286551" (at 106.68 73.025 0)
-      (effects (font (size 1.27 1.27)) hide)
-    )
+    (property "PartNumber" "NLV25T-101J-PF" (at 106.68 73.025 0)
+      (effects (font (size 1.27 1.27)) hide)
+    )
+    (property "LCSCStockCode" "C76826" (at 106.68 73.025 0)
+      (effects (font (size 1.27 1.27)) hide)
+    )
